Commit message: added datum option in navsat.xml, checked odometry drift and correction at the end of mission. Periodical surfacing disabled(something wrong with the setting)

File: alpha_rise_stonefish/description/alpha_rise.scn.xacro (robot description, xacro)
@@ -140,5 +140,5 @@
                 <link name="Base"/>
                 <origin rpy="3.1415926 0.0 0.0" xyz="-0.65 0.0 -0.05"/>
-                <noise angle="0.01745" angular_velocity="0.001745"/>
+                <noise angle="0.01 0.01 0.05" angular_velocity="0.05" yaw_drift="0.001" linear_acceleration="0.1"/>
                 <ros_publisher topic="/${robot_name}/imu/stonefish/data"/>
             </sensor>
@@ -146,7 +146,14 @@
                 <link name="Base"/>
                 <origin rpy="0.0 0.0 0.0" xyz="-0.7 0.0 -0.3"/>
-                <noise ned_position="0.5"/>
+                <noise ned_position="0.1"/>
                 <ros_publisher topic="/${robot_name}/gps/fix"/>
             </sensor>
+            <!-- <sensor name="odom" rate="10.0" type="odometry">
+                <noise position="0.00" velocity="0.00" angle="0.0" angular_velocity="0.00"/>
+                <history samples="1"/>
+                <origin xyz="0.0 0.0 0.0" rpy="3.1415926 0.0 -1.5707963"/>
+                <link name="Base"/>
+                <ros_publisher topic="/${robot_name}/sf/odometry"/>
+            </sensor> -->
             <!-- perception sensors -->
             <!-- <sensor name="mss" rate="5.0" type="profiler">

File: alpha_rise_stonefish/scenarios/ocean.scn.xacro (robot description, xacro)
@@ -10,5 +10,5 @@
     <xacro:arg name="robot_name" default="changeme"/>
     <xacro:include filename="$(find alpha_rise_stonefish)/description/alpha_rise.scn.xacro"/>
-    <xacro:alpha_rise robot_name="$(arg robot_name)" xyz="0.0 0.0 0.0" rpy="0.0 0.0 1.5707963"/>
+    <xacro:alpha_rise robot_name="$(arg robot_name)" xyz="0.0 0.0 0.0" rpy="0.0 0.0 0.0"/>
     <environment>
         <ned latitude="41" longitude="71"/>
@@ -18,5 +18,5 @@
             <particles enabled="true"/>
             <current type="uniform">
-                <velocity xyz="0.0 0.0 0.0"/>
+                <velocity xyz="0.1 0.0 0.0"/>
             </current>
             <!-- <current type="jet">
