Commit message: test

File: alpha_rise_description/urdf/base.urdf.xacro (robot description, xacro)
@@ -34,4 +34,5 @@
         <child link="pressure"/>
     </joint>
+<!--
     <link name="dvl"/>
     <joint name="dvl_joint" type="fixed">
@@ -39,5 +40,5 @@
         <parent link="base_link"/>
         <child link="dvl"/>
-    </joint>
+    </joint> -->
     <link name="surge_thruster_link"/>
     <joint name="surge_thruster_joint" type="fixed">

Commit message: localization files are included in bringup/launch/include, and alpha_rise_config. needs to edit these files

File: alpha_rise_description/urdf/base.urdf.xacro (robot description, xacro)
@@ -21,5 +21,5 @@
         <child link="imu"/>
     </joint>
-    <link name="gps"/>
+    <!-- <link name="gps"/>
     <joint name="gps_joint" type="fixed">
         <origin xyz="0.1 0.0 0.407241" rpy="3.1415 0.0 0.0"/>
@@ -30,8 +30,7 @@
     <joint name="pressure_joint" type="fixed">
         <origin xyz="-0.187845 -0.060 0.124465" rpy="0.0 3.14159265359 0.0"/>
-        <!--origin xyz="-0.087845 0.060 -0.124465" rpy="0.0 0.0 0.0"/-->
         <parent link="base_link"/>
         <child link="pressure"/>
-    </joint>
+    </joint> -->
 <!--
     <link name="dvl"/>
@@ -41,4 +40,5 @@
         <child link="dvl"/>
     </joint> -->
+<!--
     <link name="surge_thruster_link"/>
     <joint name="surge_thruster_joint" type="fixed">
@@ -63,5 +63,5 @@
         <origin xyz="0.57635 0.0 0.105" rpy="0.0 0.0 1.57079632679"/>
         <parent link="base_link"/>
-        <child link="sway_bow_thruster_link"/>
-    </joint>
+        <child link="sway_bow_thruster_link"/> -->
+    <!-- </joint> -->
 </robot>

Commit message: fixed the dvl and imu problem. all stonefish imu and dvl is appended with _sf in the frame_id

File: alpha_rise_description/urdf/base.urdf.xacro (robot description, xacro)
@@ -11,5 +11,5 @@
     <link name="cg_link"/>
     <joint name="cg_joint" type="fixed">
-        <origin xyz="0.100 0.000 0.10" rpy="3.14159265359 0.0 0.0"/>
+        <origin xyz="0.100 0.000 0.10" rpy="0.0 0.0 0.0"/>
         <parent link="base_link"/>
         <child link="cg_link"/>
@@ -17,7 +17,25 @@
     <link name="imu"/>
     <joint name="imu_joint" type="fixed">
-        <origin xyz="-0.0465 0.060 0.14648" rpy="3.14159265359 0.0 0.0"/>
+        <origin xyz="0.0 0.0 0.0" rpy="0.0 0.0 0.0"/>
         <parent link="base_link"/>
         <child link="imu"/>
+    </joint>
+    <link name="imu_sf"/>
+    <joint name="imu__sf_joint" type="fixed">
+        <origin xyz="0.0 0.0 0.0" rpy="3.1415926 0.0 0.0"/>
+        <parent link="base_link"/>
+        <child link="imu_sf"/>
+    </joint>
+    <link name="dvl"/>
+    <joint name="dvl_joint" type="fixed">
+        <origin xyz="0.0 0.0 0.0" rpy="3.1415926 0.0 0.0"/>
+        <parent link="base_link"/>
+        <child link="dvl"/>
+    </joint>
+     <link name="dvl_sf"/>
+    <joint name="dvl_sf_joint" type="fixed">
+        <origin xyz="0.0 0.0 0.0" rpy="3.1415926 0.0 0.0"/>
+        <parent link="dvl"/>
+        <child link="dvl_sf"/>
     </joint>
     <!-- <link name="gps"/>
@@ -32,11 +50,4 @@
         <parent link="base_link"/>
         <child link="pressure"/>
-    </joint> -->
-<!--
-    <link name="dvl"/>
-    <joint name="dvl_joint" type="fixed">
-        <origin xyz="0.0 0.0 0.0" rpy="0.0 0.0 0.0"/>
-        <parent link="base_link"/>
-        <child link="dvl"/>
     </joint> -->
 <!--

File: alpha_rise_stonefish/description/alpha_rise.scn.xacro (robot description, xacro)
@@ -129,5 +129,5 @@
                 <ros_publisher topic="/${robot_name}/pressure"/>
             </sensor>
-            <sensor name="dvl" type="dvl" rate="5.0">
+            <sensor name="dvl_sf" type="dvl" rate="5.0">
                 <link name="Base"/>
                 <origin rpy="3.1415926 0.0 0.0" xyz="-0.65 0.0 0.1"/>
@@ -137,5 +137,5 @@
                 <ros_publisher topic="/${robot_name}/dvl/twist" altitude_topic="/${robot_name}/dvl/altitude"/>
             </sensor>
-            <sensor name="imu" type="imu" rate="20.0">
+            <sensor name="imu_sf" type="imu" rate="20.0">
                 <link name="Base"/>
                 <origin rpy="3.1415926 0.0 0.0" xyz="-0.65 0.0 -0.05"/>
@@ -150,13 +150,13 @@
             </sensor>
             <!-- perception sensors -->
-            <!-- <sensor name="MSIS" type="msis">
-                <specs step="0.18" bins="250" horizontal_beam_width="2.0" vertical_beam_width="15.0"/>
-                <settings range_min="0.5" range_max="100.0" rotation_min="-10.0" rotation_max="10.0" gain="1.5"/>
+            <sensor name="MSIS" type="msis">
+                <specs step="0.9" bins="200" horizontal_beam_width="2.0" vertical_beam_width="15.0"/>
+                <settings range_min="0.75" range_max="50.0" rotation_min="-45.0" rotation_max="45.0" gain="2.5"/>
                 <noise multiplicative="0.02" additive="0.03"/>
                 <display colormap="hot"/>
-                <origin xyz="0.0 0.0 10.0" rpy="1.5707963 0.0 1.5707963"/>
+                <origin xyz="0.0 0.0 10.0" rpy="0.0 0.0 1.5707963"/>
                 <link name="Base"/>
                 <ros_publisher topic="/${robot_name}/MSIS/data"/>
-            </sensor> -->
+            </sensor>
             <!-- <sensor name="FLS" type="fls">
                 <specs beams="512" bins="250" horizontal_fov="120.0" vertical_fov="15.0"/>

Commit message: correctly configured the frames to be the same as the stonefish. ENU showing in RViz

File: alpha_rise_description/urdf/base.urdf.xacro (robot description, xacro)
@@ -9,9 +9,9 @@
         </visual>
     </link>
-    <link name="cg_link"/>
-    <joint name="cg_joint" type="fixed">
-        <origin xyz="0.100 0.000 0.10" rpy="0.0 0.0 0.0"/>
+    <link name="body_link"/>
+    <joint name="body_joint" type="fixed">
+        <origin xyz="0.0 0.0 0.0" rpy="3.1415926 0.0 0.0"/>
         <parent link="base_link"/>
-        <child link="cg_link"/>
+        <child link="body_link"/>
     </joint>
     <link name="imu"/>
@@ -23,5 +23,5 @@
     <link name="imu_sf"/>
     <joint name="imu__sf_joint" type="fixed">
-        <origin xyz="0.0 0.0 0.0" rpy="3.1415926 0.0 0.0"/>
+        <origin xyz="0.0 0.0 0.0" rpy="0.0 0.0 0.0"/>
         <parent link="base_link"/>
         <child link="imu_sf"/>

File: alpha_rise_stonefish/description/alpha_rise.scn.xacro (robot description, xacro)
@@ -126,5 +126,5 @@
                 <link name="Base"/>
                 <origin rpy="0.0 0.0 0.0" xyz="-1.20 0.0 0.0"/>
-                <noise pressure="5.0"/>
+                <noise pressure="2.0"/>
                 <ros_publisher topic="/${robot_name}/pressure"/>
             </sensor>
@@ -150,5 +150,5 @@
             </sensor>
             <!-- perception sensors -->
-            <sensor name="MSIS" type="msis">
+            <!-- <sensor name="MSIS" type="msis">
                 <specs step="0.9" bins="200" horizontal_beam_width="2.0" vertical_beam_width="15.0"/>
                 <settings range_min="0.75" range_max="50.0" rotation_min="-45.0" rotation_max="45.0" gain="2.5"/>
@@ -158,5 +158,5 @@
                 <link name="Base"/>
                 <ros_publisher topic="/${robot_name}/MSIS/data"/>
-            </sensor>
+            </sensor> -->
             <!-- <sensor name="FLS" type="fls">
                 <specs beams="512" bins="250" horizontal_fov="120.0" vertical_fov="15.0"/>

File: alpha_rise_stonefish/scenarios/ocean.scn.xacro (robot description, xacro)
@@ -10,5 +10,5 @@
     <xacro:arg name="robot_name" default="changeme"/>
     <xacro:include filename="$(find alpha_rise_stonefish)/description/alpha_rise.scn.xacro"/>
-    <xacro:alpha_rise robot_name="$(arg robot_name)" xyz="0.0 0.0 0.0" rpy="1.57070.0963 0.0 0.0"/>
+    <xacro:alpha_rise robot_name="$(arg robot_name)" xyz="0.0 0.0 0.0" rpy="0.0 0.0 0.0"/>
     <environment>
         <ned latitude="41" longitude="71"/>

Commit message: controller up running

File: alpha_rise_description/urdf/base.urdf.xacro (robot description, xacro)
@@ -3,5 +3,5 @@
     <link name="base_link">
         <visual>
-            <origin xyz="0.0 0.0 0.0" rpy="0.0 0.0 0.0"/>
+            <origin xyz="0.0 -0.63 -0.57" rpy="0.0 0.0 1.5707963"/>
             <geometry>
                 <mesh filename="package://alpha_rise_description/mesh/alpha_rise.stl" scale="0.001 0.001 0.001"/>
@@ -9,9 +9,9 @@
         </visual>
     </link>
-    <link name="body_link"/>
-    <joint name="body_joint" type="fixed">
+    <link name="cg_link"/>
+    <joint name="cg_joint" type="fixed">
         <origin xyz="0.0 0.0 0.0" rpy="3.1415926 0.0 0.0"/>
         <parent link="base_link"/>
-        <child link="body_link"/>
+        <child link="cg_link"/>
     </joint>
     <link name="imu"/>
@@ -29,5 +29,5 @@
     <link name="dvl"/>
     <joint name="dvl_joint" type="fixed">
-        <origin xyz="0.0 0.0 0.0" rpy="3.1415926 0.0 0.0"/>
+        <origin xyz="-0.22 0.0 -0.08" rpy="3.1415926 0.0 0.0"/>
         <parent link="base_link"/>
         <child link="dvl"/>
@@ -35,11 +35,11 @@
      <link name="dvl_sf"/>
     <joint name="dvl_sf_joint" type="fixed">
-        <origin xyz="0.0 0.0 0.0" rpy="3.1415926 0.0 0.0"/>
-        <parent link="dvl"/>
+        <origin xyz="-0.22 0.0 -0.08" rpy="0.0 0.0 0.0"/>
+        <parent link="base_link"/>
         <child link="dvl_sf"/>
     </joint>
-    <!-- <link name="gps"/>
+    <link name="gps"/>
     <joint name="gps_joint" type="fixed">
-        <origin xyz="0.1 0.0 0.407241" rpy="3.1415 0.0 0.0"/>
+        <origin xyz="0.0 0.0 0.28" rpy="3.1415 0.0 0.0"/>
         <parent link="base_link"/>
         <child link="gps"/>
@@ -47,12 +47,12 @@
     <link name="pressure"/>
     <joint name="pressure_joint" type="fixed">
-        <origin xyz="-0.187845 -0.060 0.124465" rpy="0.0 3.14159265359 0.0"/>
+        <origin xyz="-0.25 0.0 0.05" rpy="3.1415926 0.0 0.0"/>
         <parent link="base_link"/>
         <child link="pressure"/>
-    </joint> -->
-<!--
+    </joint>
+    <!-- thrusters -->
     <link name="surge_thruster_link"/>
     <joint name="surge_thruster_joint" type="fixed">
-        <origin xyz="-0.554 0.0 0.100" rpy="0.0 0.0 0.0"/>
+        <origin xyz="-0.68 0.0 0.0" rpy="0.0 0.0 0.0"/>
         <parent link="base_link"/>
         <child link="surge_thruster_link"/>
@@ -60,5 +60,5 @@
     <link name="heave_bow_thruster_link"/>
     <joint name="heave_bow_thruster_joint" type="fixed">
-        <origin xyz="0.48735 0.0 0.089" rpy="0.0 1.57079632679 0.0"/>
+        <origin xyz="0.38 0.0 0.0" rpy="0.0 1.57079632679 0.0"/>
         <parent link="base_link"/>
         <child link="heave_bow_thruster_link"/>
@@ -66,5 +66,5 @@
     <link name="heave_stern_thruster_link"/>
     <joint name="heave_stern_thruster_joint" type="fixed">
-        <origin xyz="-0.28045 0.0 0.089" rpy="0.0 1.57079632679 0.0"/>
+        <origin xyz="-0.38 0.0 0.0" rpy="0.0 1.57079632679 0.0"/>
         <parent link="base_link"/>
         <child link="heave_stern_thruster_link"/>
@@ -72,7 +72,7 @@
     <link name="sway_bow_thruster_link"/>
     <joint name="sway_bow_thruster_joint" type="fixed">
-        <origin xyz="0.57635 0.0 0.105" rpy="0.0 0.0 1.57079632679"/>
+        <origin xyz="0.48 0.0 0.0" rpy="0.0 0.0 -1.57079632679"/>
         <parent link="base_link"/>
-        <child link="sway_bow_thruster_link"/> -->
-    <!-- </joint> -->
+        <child link="sway_bow_thruster_link"/>
+    </joint>
 </robot>

Commit message: path following local working. trying global

File: alpha_rise_description/urdf/base.urdf.xacro (robot description, xacro)
@@ -76,3 +76,10 @@
         <child link="sway_bow_thruster_link"/>
     </joint>
+    <!-- perception sensors -->
+    <!-- <link name="mss"/>
+    <joint name="mss_joint" type="fixed">
+        <origin xyz="0.65 0.0 0.0" rpy="3.1415926 1.5707963 0.0"/>
+        <parent link="base_link"/>
+        <child link="mss"/>
+    </joint> -->
 </robot>

File: alpha_rise_stonefish/description/alpha_rise.scn.xacro (robot description, xacro)
@@ -33,5 +33,5 @@
                     <origin rpy="0.0 0.0 0.0" xyz="0.0 0.0 0.0"/>
                     <material name="Foam"/>
-                    <mass value="1.0"/>
+                    <mass value="1.5"/>
                     <look name="grey"/>
                     <compound_transform rpy="0.0 1.571 0.0" xyz="-0.65 0.0 -0.1"/>
@@ -150,12 +150,21 @@
             </sensor>
             <!-- perception sensors -->
-            <!-- <sensor name="MSIS" type="msis">
-                <specs step="0.9" bins="200" horizontal_beam_width="2.0" vertical_beam_width="15.0"/>
+            <!-- <sensor name="mss" rate="5.0" type="profiler">
+                <specs fov="90.0" steps="100"/>
+                <range distance_min="0.5" distance_max="100.0"/>
+                <noise distance="0.05"/>
+                <history samples="1"/>
+                <origin xyz="0.0 0.0 0.0" rpy="0.0 -1.5707963 0.0"/>
+                <link name="Base"/>
+                <ros_publisher topic="/${robot_name}/MSS/data"/>
+            </sensor> -->
+            <!-- <sensor name="msis" type="msis">
+                <specs step="1.8" bins="1250" horizontal_beam_width="2.0" vertical_beam_width="15.0"/>
                 <settings range_min="0.75" range_max="50.0" rotation_min="-45.0" rotation_max="45.0" gain="2.5"/>
                 <noise multiplicative="0.02" additive="0.03"/>
-                <display colormap="hot"/>
-                <origin xyz="0.0 0.0 10.0" rpy="0.0 0.0 1.5707963"/>
+                <display colormap="gray"/>
+                <origin xyz="0.0 0.0 0.0" rpy="0.0 0.0 1.5707963"/>
                 <link name="Base"/>
-                <ros_publisher topic="/${robot_name}/MSIS/data"/>
+                <ros_publisher topic="/${robot_name}/msis/data"/>
             </sensor> -->
             <!-- <sensor name="FLS" type="fls">

Commit message: fuse gps into odom, and convert gps into odom, track wpt in the odom frame

File: alpha_rise_description/urdf/base.urdf.xacro (robot description, xacro)
@@ -41,5 +41,5 @@
     <link name="gps"/>
     <joint name="gps_joint" type="fixed">
-        <origin xyz="0.0 0.0 0.28" rpy="3.1415 0.0 0.0"/>
+        <origin xyz="0.0 0.0 0.28" rpy="3.1415926 0.0 -1.5707963"/>
         <parent link="base_link"/>
         <child link="gps"/>

File: alpha_rise_stonefish/description/alpha_rise.scn.xacro (robot description, xacro)
@@ -134,5 +134,5 @@
                 <specs beam_angle="30.0"/>
                 <range velocity="9.0 9.0 9.0" altitude_min="0.2" altitude_max="200.0"/>
-                <noise velocity="0.0015" altitude="0.001"/>
+                <noise velocity="0.015" altitude="0.001"/>
                 <ros_publisher topic="/${robot_name}/dvl/twist" altitude_topic="/${robot_name}/dvl/altitude"/>
             </sensor>
@@ -140,5 +140,5 @@
                 <link name="Base"/>
                 <origin rpy="3.1415926 0.0 0.0" xyz="-0.65 0.0 -0.05"/>
-                <noise angle="0.000001745" angular_velocity="0.00001745"/>
+                <noise angle="0.01745" angular_velocity="0.001745"/>
                 <ros_publisher topic="/${robot_name}/imu/stonefish/data"/>
             </sensor>

File: alpha_rise_stonefish/scenarios/ocean.scn.xacro (robot description, xacro)
@@ -10,5 +10,5 @@
     <xacro:arg name="robot_name" default="changeme"/>
     <xacro:include filename="$(find alpha_rise_stonefish)/description/alpha_rise.scn.xacro"/>
-    <xacro:alpha_rise robot_name="$(arg robot_name)" xyz="0.0 0.0 0.0" rpy="0.0 0.0 0.0"/>
+    <xacro:alpha_rise robot_name="$(arg robot_name)" xyz="0.0 0.0 0.0" rpy="0.0 0.0 1.5707963"/>
     <environment>
         <ned latitude="41" longitude="71"/>

Commit message: URDF adjusted for the new rise

File: alpha_rise_description/urdf/base.urdf.xacro (robot description, xacro)
@@ -3,5 +3,5 @@
     <link name="base_link">
         <visual>
-            <origin xyz="0.0 -0.63 -0.57" rpy="0.0 0.0 1.5707963"/>
+            <origin xyz="0.0 0.0 0.0" rpy="1.5707 0.0 1.5707"/>
             <geometry>
                 <mesh filename="package://alpha_rise_description/mesh/alpha_rise.stl" scale="0.001 0.001 0.001"/>
@@ -29,5 +29,5 @@
     <link name="dvl"/>
     <joint name="dvl_joint" type="fixed">
-        <origin xyz="-0.22 0.0 -0.08" rpy="3.1415926 0.0 0.0"/>
+        <origin xyz="0.7 0.0 -0.1" rpy="3.1415926 0.0 0.0"/>
         <parent link="base_link"/>
         <child link="dvl"/>
@@ -41,5 +41,5 @@
     <link name="gps"/>
     <joint name="gps_joint" type="fixed">
-        <origin xyz="0.0 0.0 0.28" rpy="3.1415926 0.0 -1.5707963"/>
+        <origin xyz="0.45 0.0 0.28" rpy="3.1415926 0.0 0.0"/>
         <parent link="base_link"/>
         <child link="gps"/>
@@ -47,5 +47,5 @@
     <link name="pressure"/>
     <joint name="pressure_joint" type="fixed">
-        <origin xyz="-0.25 0.0 0.05" rpy="3.1415926 0.0 0.0"/>
+        <origin xyz="0.32 0.0 0.05" rpy="3.1415926 0.0 0.0"/>
         <parent link="base_link"/>
         <child link="pressure"/>
@@ -54,5 +54,5 @@
     <link name="surge_thruster_link"/>
     <joint name="surge_thruster_joint" type="fixed">
-        <origin xyz="-0.68 0.0 0.0" rpy="0.0 0.0 0.0"/>
+        <origin xyz="-0.57 0.0 0.0" rpy="0.0 0.0 0.0"/>
         <parent link="base_link"/>
         <child link="surge_thruster_link"/>
@@ -60,5 +60,5 @@
     <link name="heave_bow_thruster_link"/>
     <joint name="heave_bow_thruster_joint" type="fixed">
-        <origin xyz="0.38 0.0 0.0" rpy="0.0 1.57079632679 0.0"/>
+        <origin xyz="0.58 0.0 0.0" rpy="0.0 1.57079632679 0.0"/>
         <parent link="base_link"/>
         <child link="heave_bow_thruster_link"/>
@@ -66,5 +66,5 @@
     <link name="heave_stern_thruster_link"/>
     <joint name="heave_stern_thruster_joint" type="fixed">
-        <origin xyz="-0.38 0.0 0.0" rpy="0.0 1.57079632679 0.0"/>
+        <origin xyz="-0.18 0.0 0.0" rpy="0.0 1.57079632679 0.0"/>
         <parent link="base_link"/>
         <child link="heave_stern_thruster_link"/>
@@ -72,5 +72,5 @@
     <link name="sway_bow_thruster_link"/>
     <joint name="sway_bow_thruster_joint" type="fixed">
-        <origin xyz="0.48 0.0 0.0" rpy="0.0 0.0 -1.57079632679"/>
+        <origin xyz="0.71 0.0 0.0" rpy="0.0 0.0 -1.57079632679"/>
         <parent link="base_link"/>
         <child link="sway_bow_thruster_link"/>

File: alpha_rise_stonefish/description/alpha_rise.scn.xacro (robot description, xacro)
@@ -140,5 +140,5 @@
                 <link name="Base"/>
                 <origin rpy="3.1415926 0.0 0.0" xyz="-0.65 0.0 -0.05"/>
-                <noise angle="0.01 0.01 0.05" angular_velocity="0.05" yaw_drift="0.001" linear_acceleration="0.1"/>
+                <noise angle="0.001 0.001 0.005" angular_velocity="0.005" yaw_drift="0.001" linear_acceleration="0.001"/>
                 <ros_publisher topic="/${robot_name}/imu/stonefish/data"/>
             </sensor>
@@ -146,5 +146,5 @@
                 <link name="Base"/>
                 <origin rpy="0.0 0.0 0.0" xyz="-0.7 0.0 -0.3"/>
-                <noise ned_position="0.1"/>
+                <noise ned_position="0.0"/>
                 <ros_publisher topic="/${robot_name}/gps/fix"/>
             </sensor>

Commit message: update to tank test adjustment

File: alpha_rise_description/urdf/base.urdf.xacro (robot description, xacro)
@@ -60,5 +60,5 @@
     <link name="heave_bow_thruster_link"/>
     <joint name="heave_bow_thruster_joint" type="fixed">
-        <origin xyz="0.58 0.0 0.0" rpy="0.0 1.57079632679 0.0"/>
+        <origin xyz="0.4755 0.0 0.0" rpy="0.0 1.57079632679 0.0"/>
         <parent link="base_link"/>
         <child link="heave_bow_thruster_link"/>
@@ -66,5 +66,5 @@
     <link name="heave_stern_thruster_link"/>
     <joint name="heave_stern_thruster_joint" type="fixed">
-        <origin xyz="-0.18 0.0 0.0" rpy="0.0 1.57079632679 0.0"/>
+        <origin xyz="-0.3 0.0 0.0" rpy="0.0 1.57079632679 0.0"/>
         <parent link="base_link"/>
         <child link="heave_stern_thruster_link"/>

Commit message: update config after tank test

File: alpha_rise_description/urdf/base.urdf.xacro (robot description, xacro)
@@ -17,5 +17,5 @@
     <link name="imu"/>
     <joint name="imu_joint" type="fixed">
-        <origin xyz="0.0 0.0 0.0" rpy="0.0 0.0 0.0"/>
+        <origin xyz="0.0 0.09 0.0" rpy="0.0 0.0 0.0"/>
         <parent link="base_link"/>
         <child link="imu"/>
@@ -29,5 +29,5 @@
     <link name="dvl"/>
     <joint name="dvl_joint" type="fixed">
-        <origin xyz="0.7 0.0 -0.1" rpy="3.1415926 0.0 0.0"/>
+        <origin xyz="0.0625 0.0 -0.1" rpy="3.1415926 0.0 0.0"/>
         <parent link="base_link"/>
         <child link="dvl"/>
@@ -51,4 +51,10 @@
         <child link="pressure"/>
     </joint>
+    <link name="ping360_link"/>
+    <joint name="ping360_joint" type="fixed">
+        <origin xyz="0.792 0.0 -0.085" rpy="3.1415926 0.0 0.0"/>
+        <parent link="base_link"/>
+        <child link="ping360_link"/>
+    </joint>
     <!-- thrusters -->
     <link name="surge_thruster_link"/>
@@ -60,5 +66,5 @@
     <link name="heave_bow_thruster_link"/>
     <joint name="heave_bow_thruster_joint" type="fixed">
-        <origin xyz="0.4755 0.0 0.0" rpy="0.0 1.57079632679 0.0"/>
+        <origin xyz="0.387 0.0 0.0" rpy="0.0 1.57079632679 0.0"/>
         <parent link="base_link"/>
         <child link="heave_bow_thruster_link"/>
@@ -66,5 +72,5 @@
     <link name="heave_stern_thruster_link"/>
     <joint name="heave_stern_thruster_joint" type="fixed">
-        <origin xyz="-0.3 0.0 0.0" rpy="0.0 1.57079632679 0.0"/>
+        <origin xyz="-0.387 0.0 0.0" rpy="0.0 1.57079632679 0.0"/>
         <parent link="base_link"/>
         <child link="heave_stern_thruster_link"/>
@@ -72,5 +78,5 @@
     <link name="sway_bow_thruster_link"/>
     <joint name="sway_bow_thruster_joint" type="fixed">
-        <origin xyz="0.71 0.0 0.0" rpy="0.0 0.0 -1.57079632679"/>
+        <origin xyz="0.71 0.0 0.0" rpy="0.0 0.0 1.57079632679"/>
         <parent link="base_link"/>
         <child link="sway_bow_thruster_link"/>

Commit message: fix the MSIS tf

File: alpha_rise_description/urdf/base.urdf.xacro (robot description, xacro)
@@ -53,5 +53,5 @@
     <link name="ping360_link"/>
     <joint name="ping360_joint" type="fixed">
-        <origin xyz="0.792 0.0 -0.085" rpy="3.1415926 0.0 0.0"/>
+        <origin xyz="0.792 0.0 -0.085" rpy="3.1415926 0.0 3.1415926"/>
         <parent link="base_link"/>
         <child link="ping360_link"/>

Commit message: fix IMU tf

File: alpha_rise_description/urdf/base.urdf.xacro (robot description, xacro)
@@ -17,5 +17,5 @@
     <link name="imu"/>
     <joint name="imu_joint" type="fixed">
-        <origin xyz="0.0 0.09 0.0" rpy="0.0 0.0 0.0"/>
+        <origin xyz="0.0 -0.09 0.0" rpy="-3.1415926 0.0 3.1415926"/>
         <parent link="base_link"/>
         <child link="imu"/>
