Commit message: updated alpha_rise urdf to make imu the same as real vehicle. small changes to the localization launch file and mission config.

File: alpha_rise_description/urdf/base.urdf.xacro (robot description, xacro)
@@ -3,5 +3,5 @@
     <link name="base_link">
         <visual>
-            <origin xyz="0.0 0.0 0.0" rpy="1.5707 0.0 1.5707"/>
+            <origin xyz="-0.2 0.0 0.0" rpy="1.5707 0.0 1.5707"/>
             <geometry>
                 <mesh filename="package://alpha_rise_description/mesh/alpha_rise.stl" scale="0.001 0.001 0.001"/>
@@ -17,5 +17,5 @@
     <link name="imu"/>
     <joint name="imu_joint" type="fixed">
-        <origin xyz="0.0 -0.09 0.0" rpy="-3.1415926 0.0 3.1415926"/>
+        <origin xyz="0.0 -0.09 0.0" rpy="3.1415926 0.0 3.1415926"/>
         <parent link="base_link"/>
         <child link="imu"/>
@@ -24,5 +24,5 @@
     <joint name="imu__sf_joint" type="fixed">
         <origin xyz="0.0 0.0 0.0" rpy="0.0 0.0 0.0"/>
-        <parent link="base_link"/>
+        <parent link="imu"/>
         <child link="imu_sf"/>
     </joint>
@@ -53,5 +53,5 @@
     <link name="ping360_link"/>
     <joint name="ping360_joint" type="fixed">
-        <origin xyz="0.792 0.0 -0.085" rpy="3.1415926 0.0 3.1415926"/>
+        <origin xyz="0.592 0.0 -0.085" rpy="3.1415926 0.0 3.1415926"/>
         <parent link="base_link"/>
         <child link="ping360_link"/>
@@ -60,5 +60,5 @@
     <link name="surge_thruster_link"/>
     <joint name="surge_thruster_joint" type="fixed">
-        <origin xyz="-0.57 0.0 0.0" rpy="0.0 0.0 0.0"/>
+        <origin xyz="-0.77 0.0 0.0" rpy="0.0 0.0 0.0"/>
         <parent link="base_link"/>
         <child link="surge_thruster_link"/>
@@ -66,5 +66,5 @@
     <link name="heave_bow_thruster_link"/>
     <joint name="heave_bow_thruster_joint" type="fixed">
-        <origin xyz="0.387 0.0 0.0" rpy="0.0 1.57079632679 0.0"/>
+        <origin xyz="0.387 0.0 0.0" rpy="0.0 -1.57079632679 0.0"/>
         <parent link="base_link"/>
         <child link="heave_bow_thruster_link"/>
@@ -72,5 +72,5 @@
     <link name="heave_stern_thruster_link"/>
     <joint name="heave_stern_thruster_joint" type="fixed">
-        <origin xyz="-0.387 0.0 0.0" rpy="0.0 1.57079632679 0.0"/>
+        <origin xyz="-0.387 0.0 0.0" rpy="0.0 -1.57079632679 0.0"/>
         <parent link="base_link"/>
         <child link="heave_stern_thruster_link"/>
@@ -78,5 +78,5 @@
     <link name="sway_bow_thruster_link"/>
     <joint name="sway_bow_thruster_joint" type="fixed">
-        <origin xyz="0.71 0.0 0.0" rpy="0.0 0.0 1.57079632679"/>
+        <origin xyz="0.51 0.0 0.0" rpy="0.0 0.0 1.57079632679"/>
         <parent link="base_link"/>
         <child link="sway_bow_thruster_link"/>

Commit message: updated configuration for new mvp and electronics

File: alpha_rise_description/urdf/base.urdf.xacro (robot description, xacro)
@@ -17,5 +17,5 @@
     <link name="imu"/>
     <joint name="imu_joint" type="fixed">
-        <origin xyz="0.0 -0.09 0.0" rpy="3.1415926 0.0 3.1415926"/>
+        <origin xyz="0.0 -0.09 0.0" rpy="3.1415926 0.0 0.0"/>
         <parent link="base_link"/>
         <child link="imu"/>

Commit message: adjusted the urdf tf and the rviz model

File: alpha_rise_description/urdf/base.urdf.xacro (robot description, xacro)
@@ -1,12 +1,18 @@
 <?xml version="1.0"?>
 <robot name="alpha_rise" xmlns:xacro="http://ros.org/wiki/xacro">
-    <link name="base_link">
+    <link name="nose_tip_link">
         <visual>
-            <origin xyz="-0.2 0.0 0.0" rpy="1.5707 0.0 1.5707"/>
+            <origin xyz="00.0 0.0 0.0" rpy="0.0 0.0 0.0"/>
             <geometry>
-                <mesh filename="package://alpha_rise_description/mesh/alpha_rise.stl" scale="0.001 0.001 0.001"/>
+                <mesh filename="package://alpha_rise_description/mesh/alpha_rise_rviz.stl" scale="0.001 0.001 0.001"/>
             </geometry>
         </visual>
     </link>
+    <link name="base_link"/>
+    <joint name="base_link" type="fixed">
+        <origin xyz="0.72 0.0 0.0" rpy="0.0 0.0 0.0"/>
+        <parent link="base_link"/>
+        <child link="nose_tip_link"/>
+    </joint>
     <link name="cg_link"/>
     <joint name="cg_joint" type="fixed">
@@ -17,5 +23,5 @@
     <link name="imu"/>
     <joint name="imu_joint" type="fixed">
-        <origin xyz="0.0 -0.09 0.0" rpy="3.1415926 0.0 0.0"/>
+        <origin xyz="-0.2 -0.07 0.0" rpy="3.1415926 0.0 0.0"/>
         <parent link="base_link"/>
         <child link="imu"/>
@@ -29,5 +35,5 @@
     <link name="dvl"/>
     <joint name="dvl_joint" type="fixed">
-        <origin xyz="0.0625 0.0 -0.1" rpy="3.1415926 0.0 0.0"/>
+        <origin xyz="0.51 0.0 -0.1" rpy="3.1415926 0.0 0.0"/>
         <parent link="base_link"/>
         <child link="dvl"/>
@@ -35,5 +41,5 @@
      <link name="dvl_sf"/>
     <joint name="dvl_sf_joint" type="fixed">
-        <origin xyz="-0.22 0.0 -0.08" rpy="0.0 0.0 0.0"/>
+        <origin xyz="0.51 0.0 -0.1" rpy="0.0 0.0 0.0"/>
         <parent link="base_link"/>
         <child link="dvl_sf"/>
@@ -41,5 +47,5 @@
     <link name="gps"/>
     <joint name="gps_joint" type="fixed">
-        <origin xyz="0.45 0.0 0.28" rpy="3.1415926 0.0 0.0"/>
+        <origin xyz="0.05 0.0 0.32" rpy="3.1415926 0.0 0.0"/>
         <parent link="base_link"/>
         <child link="gps"/>
@@ -47,5 +53,5 @@
     <link name="pressure"/>
     <joint name="pressure_joint" type="fixed">
-        <origin xyz="0.32 0.0 0.05" rpy="3.1415926 0.0 0.0"/>
+        <origin xyz="0.3 0.0 0.05" rpy="3.1415926 0.0 0.0"/>
         <parent link="base_link"/>
         <child link="pressure"/>
@@ -53,5 +59,5 @@
     <link name="ping360_link"/>
     <joint name="ping360_joint" type="fixed">
-        <origin xyz="0.592 0.0 -0.085" rpy="3.1415926 0.0 3.1415926"/>
+        <origin xyz="0.63 0.0 -0.085" rpy="0.0 0.0 3.1415926"/>
         <parent link="base_link"/>
         <child link="ping360_link"/>
@@ -72,5 +78,5 @@
     <link name="heave_stern_thruster_link"/>
     <joint name="heave_stern_thruster_joint" type="fixed">
-        <origin xyz="-0.387 0.0 0.0" rpy="0.0 -1.57079632679 0.0"/>
+        <origin xyz="-0.4 0.0 0.0" rpy="0.0 -1.57079632679 0.0"/>
         <parent link="base_link"/>
         <child link="heave_stern_thruster_link"/>

Commit message: feat: add ping360_sf_link

File: alpha_rise_description/urdf/base.urdf.xacro (robot description, xacro)
@@ -63,4 +63,10 @@
         <child link="ping360_link"/>
     </joint>
+    <link name="ping360_link_sf"/>
+    <joint name="ping360_sf_joint" type="fixed">
+        <origin xyz="0.63 0.0 -0.085" rpy="0.0 0.0 0"/>
+        <parent link="base_link"/>
+        <child link="ping360_link_sf"/>
+    </joint>
     <!-- thrusters -->
     <link name="surge_thruster_link"/>

Commit message: fix:ping360_sf link

File: alpha_rise_description/urdf/base.urdf.xacro (robot description, xacro)
@@ -65,5 +65,5 @@
     <link name="ping360_link_sf"/>
     <joint name="ping360_sf_joint" type="fixed">
-        <origin xyz="0.63 0.0 -0.085" rpy="0.0 0.0 0"/>
+        <origin xyz="0.0 0.0 -0.0" rpy="3.14 0.0 0.0"/>
         <parent link="base_link"/>
         <child link="ping360_link_sf"/>

Commit message: updated launch files for field test

File: alpha_rise_description/urdf/base.urdf.xacro (robot description, xacro)
@@ -47,5 +47,5 @@
     <link name="gps"/>
     <joint name="gps_joint" type="fixed">
-        <origin xyz="0.05 0.0 0.32" rpy="3.1415926 0.0 0.0"/>
+        <origin xyz="0.05 0.0 0.32" rpy="0.0 0.0 0.0"/>
         <parent link="base_link"/>
         <child link="gps"/>
@@ -65,5 +65,5 @@
     <link name="ping360_link_sf"/>
     <joint name="ping360_sf_joint" type="fixed">
-        <origin xyz="0.0 0.0 -0.0" rpy="3.14 0.0 0.0"/>
+        <origin xyz="0.63 0.0 -0.085" rpy="3.14 0.0 0.0"/>
         <parent link="base_link"/>
         <child link="ping360_link_sf"/>

Commit message: 08-23 config

File: alpha_rise_description/urdf/base.urdf.xacro (robot description, xacro)
@@ -23,5 +23,5 @@
     <link name="imu"/>
     <joint name="imu_joint" type="fixed">
-        <origin xyz="-0.2 -0.07 0.0" rpy="3.1415926 0.0 0.0"/>
+        <origin xyz="-0.2 -0.0 0.0" rpy="0 0.0 0.0"/>
         <parent link="base_link"/>
         <child link="imu"/>

Commit message: fixed simulation issue for IMU

File: alpha_rise_description/urdf/base.urdf.xacro (robot description, xacro)
@@ -29,5 +29,5 @@
     <link name="imu_sf"/>
     <joint name="imu__sf_joint" type="fixed">
-        <origin xyz="0.0 0.0 0.0" rpy="0.0 0.0 0.0"/>
+        <origin xyz="0.0 0.0 0.0" rpy="3.1415926 0.0 0.0"/>
         <parent link="imu"/>
         <child link="imu_sf"/>

Commit message: change to the AUV imu joint to improve accuracy of localization for inter-world transform

File: alpha_rise_description/urdf/base.urdf.xacro (robot description, xacro)
@@ -23,6 +23,6 @@
     <link name="imu"/>
     <joint name="imu_joint" type="fixed">
-        <origin xyz="-0.2 -0.0 0.0" rpy="0 0.0 0.0"/>
-        <parent link="base_link"/>
+        <origin xyz="-0.65 0.0 0.05" rpy="0 0.0 0.0"/>
+        <parent link="nose_tip_link"/>
         <child link="imu"/>
     </joint>
@@ -47,6 +47,7 @@
     <link name="gps"/>
     <joint name="gps_joint" type="fixed">
-        <origin xyz="0.05 0.0 0.32" rpy="0.0 0.0 0.0"/>
-        <parent link="base_link"/>
+        <!-- <origin xyz="0.05 0.0 0.32" rpy="0.0 0.0 0.0"/> -->
+        <origin xyz="-0.65 0.0 0.3" rpy="0.0 0.0 0.0"/>
+        <parent link="nose_tip_link"/>
         <child link="gps"/>
     </joint>
@@ -68,4 +69,18 @@
         <parent link="base_link"/>
         <child link="ping360_link_sf"/>
+    </joint>
+    <link name="HydromeaUVX"/>
+    <joint name="HydromeaUVX_joint" type="fixed">
+        <!-- <origin xyz="-0.35 0.00 0.15" rpy="0.5236 0.0 0.0"/> -->
+        <origin xyz="-0.35 0.00 -0.15" rpy="0.0 0.0 0.0"/>
+        <parent link="base_link"/>
+        <child link="HydromeaUVX"/>
+    </joint>
+    <link name="usbl_transp"/>
+    <joint name="usbl_transp_joint" type="fixed">
+        <origin xyz="0.15 0.00 -0.15" rpy="0.0 0.0 0.0"/>
+        <!-- <origin xyz="-0.5 0.00 -0.15" rpy="1.0472 0.0 0.0"/> -->
+        <parent link="base_link"/>
+        <child link="usbl_transp"/>
     </joint>
     <!-- thrusters -->

Commit message: auv demo path + updated pid parameter names + optical modem joint

File: alpha_rise_description/urdf/base.urdf.xacro (robot description, xacro)
@@ -72,6 +72,7 @@
     <link name="HydromeaUVX"/>
     <joint name="HydromeaUVX_joint" type="fixed">
+        <origin xyz="-0.35 0.00 0.15" rpy="1.5708 5.2360 1.5708 "/>
         <!-- <origin xyz="-0.35 0.00 0.15" rpy="0.5236 0.0 0.0"/> -->
-        <origin xyz="-0.35 0.00 -0.15" rpy="0.0 0.0 0.0"/>
+        <!-- <origin xyz="-0.35 0.00 -0.15" rpy="0.0 0.0 0.0"/> -->
         <parent link="base_link"/>
         <child link="HydromeaUVX"/>

Commit message: test sim changes

File: alpha_rise_description/urdf/base.urdf.xacro (robot description, xacro)
@@ -73,6 +73,4 @@
     <joint name="HydromeaUVX_joint" type="fixed">
         <origin xyz="-0.35 0.00 0.15" rpy="1.5708 5.2360 1.5708 "/>
-        <!-- <origin xyz="-0.35 0.00 0.15" rpy="0.5236 0.0 0.0"/> -->
-        <!-- <origin xyz="-0.35 0.00 -0.15" rpy="0.0 0.0 0.0"/> -->
         <parent link="base_link"/>
         <child link="HydromeaUVX"/>
